Commit message: Updated simulated hand xacro the match the changes in the frames in the palm

File: robotiq_s_model_visualization/cfg/robotiq_hand_macro.urdf.xacro (robot description, xacro)
@@ -12,14 +12,14 @@
     <link name="${prefix}link_0">
       <visual>
-        <origin xyz="0 0 0" rpy="0 0 0"/>
+        <origin xyz="0.020 0 0" rpy="0 0 0"/>
         <geometry>
           <mesh filename="package://robotiq_s_model_visualization/meshes/s-model_articulated/visual/link_0.STL" />
         </geometry>
-        <material name="green">
-          <color rgba="0 1 0 1"/>
+        <material name="gray">
+          <color rgba="0.2 0.2 0.2 1"/>
         </material>
       </visual>
       <collision>
-        <origin rpy="0 0 0" xyz="0 0 0"/>
+        <origin xyz="0.020 0 0" rpy="0 0 0"/>
         <geometry>
           <mesh filename="package://robotiq_s_model_visualization/meshes/s-model_articulated/collision/link_0.STL" />
@@ -42,18 +42,16 @@
     <link name="${prefix}link_1">
       <visual>
-        <origin rpy="0 0 ${3.1416/2}" xyz="0 0.05717 0"/>
+        <origin xyz="0.050 -.028 0" rpy="0 0 -0.52"/>
         <geometry>
           <mesh filename="package://robotiq_s_model_visualization/meshes/s-model_articulated/visual/link_1.STL" />
         </geometry>
-        <material name="green"/>
-      </visual>
-      <collision>
-        <origin rpy="0 0 ${3.1416/2}" xyz="0 0.05717 0"/>
-        <geometry>
-          <mesh filename="package://robotiq_s_model_visualization/meshes/s-model_articulated/collision/link_1.STL"/>
-        </geometry>
-        <material name="yellow">
-          <color rgba="0 1 1 1"/>
-        </material>
+        <material name="gray"/>
+      </visual>
+      <collision>
+        <origin xyz="0.050 -.028 0" rpy="0 0 -0.52"/>
+        <geometry>
+          <mesh filename="package://robotiq_s_model_visualization/meshes/s-model_articulated/collision/link_1.STL" />
+        </geometry>
+        <material name="yellow"/>
       </collision>
       <inertial>
@@ -74,16 +72,21 @@
     <!-- Link 2 -->
     <link name="${prefix}link_2">
-      <visual>
-        <origin rpy="0 0 ${3.1416/2}" xyz="0 0.03810 0.0075"/>
+      <!--
+      NOTE: This link has an offset in the z-direction based on the models that were
+      used to generate grap-it poses.  With the offset below the model appears visually
+      correct, but it is suspect.
+      -->
+      <visual>
+        <origin xyz="0.039 0 0.0075" rpy="0 0 0"/>
         <geometry>
           <mesh filename="package://robotiq_s_model_visualization/meshes/s-model_articulated/visual/link_2.STL" />
         </geometry>
-        <material name="green"/>
-      </visual>
-      <collision>
-        <origin rpy="0 0 ${3.1416/2}" xyz="0 0.03810 0.0075"/>
-          <geometry>
-            <mesh filename="package://robotiq_s_model_visualization/meshes/s-model_articulated/collision/link_2.STL"/>
-          </geometry>
+        <material name="gray"/>
+      </visual>
+      <collision>
+        <origin xyz="0.039 0 0.0075" rpy="0 0 0"/>
+        <geometry>
+          <mesh filename="package://robotiq_s_model_visualization/meshes/s-model_articulated/collision/link_2.STL" />
+        </geometry>
         <material name="yellow"/>
       </collision>
@@ -106,14 +109,14 @@
     <link name="${prefix}link_3">
       <visual>
-        <origin xyz="0 0 0" rpy="0 0 0"/>
+        <origin xyz="0 0 0" rpy="0 0 0.52"/>
         <geometry>
           <mesh filename="package://robotiq_s_model_visualization/meshes/s-model_articulated/visual/link_3.STL" />
         </geometry>
-        <material name="green"/>
-      </visual>
-      <collision>
-        <origin xyz="0 0 0" rpy="0 0 0"/>
-        <geometry>
-          <mesh filename="package://robotiq_s_model_visualization/meshes/s-model_articulated/collision/link_3.STL"/>
+        <material name="gray"/>
+      </visual>
+      <collision>
+        <origin xyz="0 0 0" rpy="0 0 0.52"/>
+        <geometry>
+          <mesh filename="package://robotiq_s_model_visualization/meshes/s-model_articulated/collision/link_3.STL" />
         </geometry>
         <material name="yellow"/>
@@ -162,4 +165,5 @@
       <mu1>1.1</mu1>
       <mu2>1.1</mu2>
+      <material>Gazebo/Red</material>
     </gazebo>
     <!-- Link paraproximal actuating hinge -->
@@ -192,4 +196,5 @@
       <mu1>1.1</mu1>
       <mu2>1.1</mu2>
+      <material>Gazebo/Red</material>
     </gazebo>
     <!-- Link proximal actuating bar -->
@@ -221,4 +226,5 @@
       <mu1>1.1</mu1>
       <mu2>1.1</mu2>
+      <material>Gazebo/Red</material>
     </gazebo>
     <!-- Link paraproximal bar -->
@@ -250,4 +256,5 @@
       <mu1>1.1</mu1>
       <mu2>1.1</mu2>
+      <material>Gazebo/Red</material>
     </gazebo>
     <!-- Link median actuating hinge -->
@@ -279,4 +286,5 @@
       <mu1>1.1</mu1>
       <mu2>1.1</mu2>
+      <material>Gazebo/Red</material>
     </gazebo>
     <!-- Link median bar -->
@@ -308,4 +316,5 @@
       <mu1>1.1</mu1>
       <mu2>1.1</mu2>
+      <material>Gazebo/Red</material>
     </gazebo>
     <!-- Link paramedian hinge -->
@@ -337,4 +346,5 @@
       <mu1>1.1</mu1>
       <mu2>1.1</mu2>
+      <material>Gazebo/Red</material>
     </gazebo>
     <!-- Link median bar underactuated -->
@@ -366,4 +376,5 @@
       <mu1>1.1</mu1>
       <mu2>1.1</mu2>
+      <material>Gazebo/Red</material>
     </gazebo>
     <!-- Link paradistal hinge -->
@@ -395,4 +406,5 @@
       <mu1>1.1</mu1>
       <mu2>1.1</mu2>
+      <material>Gazebo/Red</material>
     </gazebo>
     <!-- End of link list -->
@@ -403,6 +415,6 @@
       <child link="${prefix}link_proximal_actuating_hinge"/>
       <axis xyz="0 0 1"/>
-      <origin rpy="0 0 -2.0906" xyz="0 0 0.01"/>
-      <limit effort="100" lower="-3.1416" upper="3.1416" velocity="100"/>
+      <origin rpy="0 0 -2.0906" xyz="0.02 0 0.01"/>
+      <limit effort="0.6100" lower="-3.1416" upper="3.1416" velocity="0.0100"/>
     </joint>
     <gazebo reference="${prefix}joint_proximal_actuating_hinge">
@@ -414,5 +426,5 @@
       <child link="${prefix}link_paraproximal_actuating_hinge"/>
       <axis xyz="0 0 1"/>
-      <origin rpy="0 0 -2.0906" xyz="0 0 -0.01"/>
+      <origin rpy="0 0 -2.0906" xyz="0.02 0 -0.01"/>
       <limit effort="100" lower="-3.1416" upper="3.1416" velocity="100"/>
     </joint>
@@ -447,5 +459,5 @@
       <child link="${prefix}link_median_actuating_hinge"/>
       <axis xyz="0 0 1"/>
-      <origin rpy="0 0 ${-0.37}" xyz="0 0.05715 0.01"/>
+      <origin rpy="0 0 ${-0.37-2.0906}" xyz="0.05 -0.028 0.01"/>
       <limit effort="100" lower="-3.1416" upper="3.1416" velocity="100"/>
     </joint>
@@ -459,5 +471,5 @@
       <axis xyz="0 0 1"/>
       <!-- -0.37 is hand picked, 0.9719 is hand calculated from atan(0.02381/0.01625) -->
-      <origin rpy="0 0 0" xyz="0 0.05715 -0.01"/>
+      <origin rpy="0 0 -2.0906" xyz="0.05 -0.028 -0.01"/>
       <limit effort="100" lower="-3.1416" upper="3.1416" velocity="100"/>
     </joint>
@@ -482,5 +494,5 @@
       <child link="${prefix}link_paradistal_hinge"/>
       <axis xyz="0 0 1"/>
-      <origin rpy="0 0 0" xyz="0 0.039 -0.01"/>
+      <origin rpy="0 0 0" xyz="0.039 0 -0.01"/>
       <limit effort="100" lower="-3.1416" upper="3.1416" velocity="100"/>
     </joint>
@@ -502,5 +514,5 @@
     <!-- Joint 1 -->
     <joint name="${prefix}joint_1" type="revolute">
-      <origin rpy="0 0 -2.0906" xyz="0 0 0"/>
+      <origin xyz="0.020 0 0" rpy="0 0 0"/>
       <axis xyz="0 0 1" />
       <parent link="${prefix}link_0"/>
@@ -519,5 +531,5 @@
       <dynamics damping="1" friction="0" />
       <axis xyz="0 0 1"/>
-      <origin rpy="0 0 0" xyz="0 0.05715 0"/>
+      <origin xyz="0.050 -.028 0" rpy="0 0 -0.52"/>
       <!-- Limits: [0deg.,90deg.] -->
       <limit lower="0" upper="1.5708" effort="60" velocity="-1"/>
@@ -532,5 +544,5 @@
       <dynamics damping="1" friction="0" />
       <axis xyz="0 0 1"/>
-      <origin rpy="0 0 ${3.1416/2 + 0.5198}" xyz="0 0.039 0"/>
+      <origin xyz="0.039 0 0" rpy="0 0 0"/>
       <!-- Limits: [-38deg.,60deg.] -->
       <limit lower="-0.6632" upper="1.0471" effort="60" velocity="-1"/>
@@ -650,7 +662,5 @@
             <mesh filename="package://robotiq_s_model_visualization/meshes/s-model_articulated/visual/palm.STL" />
           </geometry>
-          <material name="green">
-            <color rgba="0 1 0 1"/>
-          </material>
+          <material name="gray"/>
         </visual>
         <!-- Simple shape collision -->
@@ -674,4 +684,5 @@
         <mu2>1.1</mu2>
       </gazebo>
+      <link name="${prefix}tool0"/>
     <!-- End of link list -->
     <!-- Joint list -->
@@ -684,5 +695,5 @@
       <origin rpy="0 3.1416 -1.57" xyz="-0.0455 0.0214 0.036"/>
       <!-- Limits: [-17deg.,17deg.] -->
-      <limit lower="-0.2967" upper="0.2967" effort="60" velocity="-1"/>
+      <limit lower="-0.2967" upper="0.2967" effort="0.6" velocity="0.001"/>
     </joint>
     <gazebo reference="${prefix}palm_finger_1_joint">
@@ -697,5 +708,5 @@
       <origin rpy="0 3.1416 -1.57" xyz="-0.0455 0.0214 -0.036"/>
       <!-- Limits: [-17deg.,17deg.] -->
-      <limit lower="-0.2967" upper="0.2967" effort="60" velocity="-1"/>
+      <limit lower="-0.2967" upper="0.2967" effort="0.6" velocity="0.001"/>
     </joint>
     <gazebo reference="${prefix}palm_finger_2_joint">
@@ -709,9 +720,14 @@
       <axis xyz="0 1 0"/>
       <origin rpy="0 0 1.57" xyz="0.0455 0.0214 0"/>
-      <limit lower="0" upper="0" effort="60" velocity="-1"/>
+      <limit lower="0" upper="0" effort="0.6" velocity="0.001"/>
     </joint>
     <gazebo reference="${prefix}palm_finger_middle_joint">
       <implicitSpringDamper>1</implicitSpringDamper>
     </gazebo>
+    <joint name="${prefix}palm_tool0" type="fixed">
+      <parent link="${prefix}palm"/>
+      <child link="${prefix}tool0"/>
+      <origin xyz="0.0 0.0875 0.0" rpy="0 0 1.5707"/>
+    </joint>
     <!-- end of joint list -->
   </xacro:macro>

File: robotiq_s_model_visualization/cfg/s-model_articulated_macro.xacro (robot description, xacro)
@@ -1,2 +1,3 @@
+<?xml version="1.0"?>
 <!--
 s-model_articulated_macro(prefix)
@@ -8,7 +9,7 @@
 	<xacro:include filename="$(find robotiq_s_model_visualization)/cfg/s-model_finger_articulated_macro.xacro" />
 	<xacro:macro name="s-model_articulated" params="prefix">
-	<xacro:s-model_finger_articulated prefix="${prefix}finger_1_"/>
-	<xacro:s-model_finger_articulated prefix="${prefix}finger_2_"/>
-	<xacro:s-model_finger_articulated prefix="${prefix}finger_middle_"/>
+		<xacro:s-model_finger_articulated prefix="${prefix}finger_1_"/>
+		<xacro:s-model_finger_articulated prefix="${prefix}finger_2_"/>
+		<xacro:s-model_finger_articulated prefix="${prefix}finger_middle_"/>
 		<!-- link list -->
 		<link name="${prefix}palm">

File: robotiq_s_model_visualization/cfg/s-model_finger_articulated_macro.xacro (robot description, xacro)
@@ -1,2 +1,3 @@
+<?xml version="1.0"?>
 <!--
 s-model_finder_articulated_macro(prefix)
@@ -108,5 +109,5 @@
 			<axis xyz="0 0 1"/>
 			<origin xyz="0.020 0 0" rpy="0 0 0"/>
-			<limit lower="0.0495" upper="1.2218" effort="100" velocity="100"/>
+			<limit lower="0.0495" upper="1.2218" effort="0.001" velocity="0.001"/>
 		</joint>
 		<joint name="${prefix}joint_2" type="revolute">
@@ -115,5 +116,5 @@
 			<axis xyz="0 0 1"/>
 			<origin xyz="0.050 -.028 0" rpy="0 0 -0.52"/>
-			<limit lower="0.0" upper="1.5708" effort="100" velocity="100"/>
+			<limit lower="0.0" upper="1.5708" effort="0.001" velocity="0.001"/>
 		</joint>
 		<joint name="${prefix}joint_3" type="revolute">
@@ -122,5 +123,5 @@
 			<axis xyz="0 0 1"/>
 			<origin xyz="0.039 0 0" rpy="0 0 0"/>
-			<limit lower="-1.2217" upper="-0.0523" effort="100" velocity="100"/>
+			<limit lower="-1.2217" upper="-0.0523" effort="0.001" velocity="0.001"/>
 		</joint>
 		<!-- end of joint list -->
